Commit message: replace inclined plane examples with URDFs

File: test/urdf/shallow_incline.urdf (robot description, URDF)
Before this commit: robot box_in_a_box, 4 links, 3 joints
Links:
- removed link floor
- removed link left_wall
- removed link right_wall
- added link plane; collision box size=4 1 0.1; collision plane normal=0 0 1
Joints:
- removed joint floor_to_box
- removed joint floor_to_left_wall
- removed joint floor_to_right_wall
- added joint plane_to_box: type planar, parent plane, child box, axis 0 1 0

File: test/urdf/steep_incline.urdf (robot description, URDF)
Before this commit: robot box_in_a_box, 4 links, 3 joints
Links:
- removed link floor
- removed link left_wall
- removed link right_wall
- added link plane; collision box size=4 1 0.1; collision plane normal=0 0 1
Joints:
- removed joint floor_to_box
- removed joint floor_to_left_wall
- removed joint floor_to_right_wall
- added joint plane_to_box: type planar, parent plane, child box, axis 0 1 0
